File: MQ4_Kicad/Esp32_C3_WROOM-02.kicad_sch (KiCad schematic)
At the start: 12 parts, among them SW1 SW_SPST, SW2 SW_SPST, U6 ESP32-C3-WROOM-02

Commit message: Ajustes 3
Connections:
- net 3,3V: no longer C13.1, C14.1, U6.1 (3V3)
- new net +3.3V: C13.1, C14.1, U6.1 (3V3)
