File: MQ4_Kicad/MQ4.kicad_sch (KiCad schematic)
At the start: 4 parts, among them J1 Motor_2, J2 Motor_4, J3 Motor_1, J4 Motor_3

Commit message: Avance de esquematicos
Parts:
- added J6: Battery_input, Connector_Molex:Molex_KK-254_AE-6410-02A_1x02_P2.54mm_Vertical, symbol Connector_Generic:Conn_01x02
- J1, J2, J3, J4: footprint (none) -> Connector_Molex:Molex_KK-254_AE-6410-02A_1x02_P2.54mm_Vertical
Connections:
- net DRV8871-3/OUT2: now reaches J3.1 (Pin_1)
- net DRV8871-3/OUT1: now reaches J3.2 (Pin_2)
- net DRV8871-4/OUT2: now reaches J4.1 (Pin_1)
- net DRV8871-4/OUT1: now reaches J4.2 (Pin_2)
- net DRV8871-1/OUT1: now reaches J1.1 (Pin_1)
- net DRV8871-1/OUT2: now reaches J1.2 (Pin_2)
- net DRV8871-2/OUT1: now reaches J2.1 (Pin_1)
- net DRV8871-2/OUT2: now reaches J2.2 (Pin_2)
- new net BAT+: J6.2 (Pin_2)
- new net GND: J6.1 (Pin_1)
- no-connect marks 0 -> 1
Other:
- removed sheet Alimentacion
- removed sheet PCB_carrito
- added sheet AP63203 (AP60203.kicad_sch)
- added sheet DRV8871-1 (DRV8871.kicad_sch)
- added sheet DRV8871-2 (DRV8871.kicad_sch)
- added sheet DRV8871-3 (DRV8871.kicad_sch)
- added sheet DRV8871-4 (DRV8871.kicad_sch)
- added sheet Esp32 C3 WROOM-02 (Esp32_C3_WROOM-02.kicad_sch)
- moved on the sheet: J1, J2, J3, J4

Commit message: Avance de esquematicos
Parts:
- added D2: PMEG6010CEH, Diode_SMD:D_SOD-123F, symbol Diode:PMEG6010CEH
- added U5: LD1117S33TR_SOT223, Package_TO_SOT_SMD:SOT-223-3_TabPin2, symbol Regulator_Linear:LD1117S33TR_SOT223
Other:
- sheet AP63203 renamed AP63205
- added sheet USB-C (usbc.kicad_sch)
- sheet AP63205 ports: added 5V; removed 3.3V

Commit message: Ajustes
Parts:
- added C18: 1uF, Capacitor_SMD:C_0805_2012Metric, symbol Device:C
- added C19: 4.7uF, Capacitor_SMD:C_0805_2012Metric, symbol Device:C
- added D3: SMD22PL, Diode_SMD:D_SOD-123F, symbol Diode:PMEG6010CEH
- D2: value PMEG6010CEH -> SMD22PL
Connections:
- net +5V: now also D3.2 (A)
- net GND: now also U5.1 (GND), C18.2, C19.2
- net +3.3V: now reaches U5.2 (VO)
- net +3.3V: now also C19.1
- net at U5.3 (VI): now also D2.1 (K), C18.1, D3.1 (K)
- net +5VUSB: now reaches D2.2 (A)
- net BAT+ renamed VBAT
Other:
- added sheet HC-SR04 (HC_SR04.kicad_sch)
- added sheet Led RGB Prog. (RGBLED.kicad_sch)
- moved on the sheet: D2, J6, U5

Commit message: Ajustes 2
Parts:
- added J8: Conn_01x03, symbol Connector_Generic:Conn_01x03
Connections:
- net +5V: now also J8.1 (Pin_1)
- net GND: now also J8.3 (Pin_3)
- new net RGB_DOUT4: J8.2 (Pin_2)
Other:
- added sheet Led RGB Prog.1 (RGBLED.kicad_sch)
- added sheet Led RGB Prog.2 (RGBLED.kicad_sch)
- added sheet Led RGB Prog.3 (RGBLED.kicad_sch)
- moved on the sheet: J1, J6

Commit message: Ajustes 3
Parts:
- removed C18: 1uF, Capacitor_SMD:C_0805_2012Metric, symbol Device:C
- removed C19: 4.7uF, Capacitor_SMD:C_0805_2012Metric, symbol Device:C
- removed D2, D3: SMD22PL, Diode_SMD:D_SOD-123F, symbol Diode:PMEG6010CEH
- removed U5: LD1117S33TR_SOT223, Package_TO_SOT_SMD:SOT-223-3_TabPin2, symbol Regulator_Linear:LD1117S33TR_SOT223
Other:
- added sheet LDL1117 (LDL1117.kicad_sch)
- sheet AP63205 ports: added none; removed 5V, GND, Vin
- sheet DRV8871-1 ports: added none; removed GND, Vin
- sheet DRV8871-2 ports: added none; removed GND, Vin
- sheet DRV8871-3 ports: added none; removed GND, Vin
- sheet DRV8871-4 ports: added none; removed GND, Vin
- sheet Esp32 C3 WROOM-02 ports: added none; removed 3,3V, GND
- sheet USB-C ports: added none; removed 5V, GND
- note added: "3.3V"
- note added: "5V"
- moved on the sheet: J6
