File: MQ4_Kicad/usbc.kicad_sch (KiCad schematic)
At the start: 11 parts, among them J5 USB_C_Receptacle_USB2.0_16P, U7 USBLC6-2SC6

Commit message: Ajustes
Parts:
- removed R14: 33, Resistor_SMD:R_0805_2012Metric, symbol Device:R
- removed R9: 5.1k, Resistor_SMD:R_0805_2012Metric_Pad1.20x1.40mm_HandSolder, symbol Device:R
- added C15: 100nF, Capacitor_SMD:C_0805_2012Metric, symbol Device:C
- added R12: 33, Resistor_SMD:R_0805_2012Metric, symbol Device:R
- renumbered C15 to C16, C16 to C17, R11 to R10, R12 to R11, R10 to R9
Connections:
- net D+: now also U7.3 (I/O2)
- net D-: now also U7.1 (I/O1); no longer R13.1
- net GND: now also J5.S1 (SHIELD), C15.2
- net USB_D+: now also R13.2; no longer U7.4 (I/O2)
- net USB_D-: now also R12.2; no longer U7.6 (I/O1)
- net at C16.1, D1.1 (K), J5.A4 (VBUS)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: now also U7.5 (VBUS), C15.1
- new net R+: R13.1, U7.4 (I/O2)
- new net R-: R12.1, U7.6 (I/O1)
- no-connect marks 3 -> 2
Other:
- moved on the sheet: C16, C17, D1, J5, R10, R11, R9, U7

Commit message: Ajustes 3
Connections:
- net 5V renamed +5VUSB
Changed lines of the file:
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@@
+	(wire
+		(pts
+			(xy 107.95 30.48) (xy 105.41 30.48)
+		)
+		(stroke
+			(width 0)
+			(type default)
+		)
+	)
 	(wire
 		(pts
@@
 		(pts
 			(xy 46.99 85.09) (xy 46.99 83.82)
+		)
+		(stroke
+			(width 0)
+			(type default)
+		)
+	)
+	(wire
+		(pts
+			(xy 107.95 34.29) (xy 107.95 30.48)
 		)
 		(stroke
@@
 		(shape bidirectional)
 		(at 113.03 59.69 0)
-		(effects
-			(font
-				(size 1.27 1.27)
-			)
-			(justify left)
-		)
-	)
-	(hierarchical_label "5V"
-		(shape output)
-		(at 107.95 34.29 0)
-		(effects
-			(font
-				(size 1.27 1.27)
-			)
-			(justify left)
-		)
-	)
-	(hierarchical_label "GND"
-		(shape input)
-		(at 49.53 83.82 0)
 		(effects
 			(font
@@
 	)
 	(symbol
+		(lib_id "power:+5VD")
+		(at 105.41 30.48 0)
+		(unit 1)
+		(body_style 1)
+		(exclude_from_sim no)
+		(in_bom yes)
+		(on_board yes)
+		(in_pos_files yes)
+		(dnp no)
+		(property "Reference" "#PWR057"
+			(at 105.41 34.29 0)
+			(hide yes)
+			(show_name no)
+			(do_not_autoplace no)
+			(effects
+				(font
+					(size 1.27 1.27)
+				)
+			)
+		)
+		(property "Value" "+5VUSB"
+			(at 105.41 26.67 0)
+			(show_name no)
+			(do_not_autoplace no)
+			(effects
+				(font
+					(size 1.27 1.27)
+				)
+			)
+		)
+		(property "Footprint" ""
+			(at 105.41 30.48 0)
+			(hide yes)
+			(show_name no)
+			(do_not_autoplace no)
+			(effects
+				(font
+					(size 1.27 1.27)
+				)
+			)
+		)
+		(property "Datasheet" ""
+			(at 105.41 30.48 0)
+			(hide yes)
+			(show_name no)
+			(do_not_autoplace no)
+			(effects
+				(font
+					(size 1.27 1.27)
+				)
+			)
+		)
+		(property "Description" "Power symbol creates a global label with name \"+5VD\""
+			(at 105.41 30.48 0)
+			(hide yes)
+			(show_name no)
+			(do_not_autoplace no)
+			(effects
+				(font
+					(size 1.27 1.27)
+				)
+			)
+		)
+		(pin "1"
+		)
+		(instances
+			(project "MQ4"
+				(path "/3122b748-b18a-4430-81c9-b624cd1e321d/9cfcb68a-848e-4404-a2cf-d894e67851b1"
+					(reference "#PWR057")
+					(unit 1)
+				)
+			)
+		)
+	)
+	(symbol
 		(lib_id "power:GND")
 		(at 76.2 53.34 0)
@@
 	(group "usbc"
 		(lib_id "USB-C 16P:usbc")
-		(members "00c08014-d9a6-458d-a25f-47aee30f3706" "05e1108e-6ade-45b6-8ee5-93297f0809cb"
-			"091f30f1-b649-4f01-b896-58e05a611ba3" "094b194e-0616-4f11-b99c-011bcc3eb3d5"
-			"0d7bf8cc-763c-4d73-a79d-c008511989c4" "1030fe69-ed03-412a-a121-e00c15f2cbd9"
-			"11be32db-d326-4050-896b-7b42c8180973" "1525eefc-db0f-4128-b1fe-bcf595bb1ef8"
-			"1763a40e-1121-4ab1-a1e8-7f43c30ca1c7" "1b906849-1e54-4e2a-93c0-fe6b986ff8b7"
-			"221f80ae-7cc2-43bf-a861-1c55bf3d46d6" "2303f457-5b0d-4715-9218-4f59bb6d9517"
-			"27a712fc-486f-424f-8355-7e1d4657289e" "2ed12085-8670-4206-8ce0-7281c614a2e6"
-			"30cca68c-2bc3-4d30-bad8-ec9e12f7a6fb" "3203af40-4d93-4104-aeb6-ea5d71acfc20"
-			"3290ba86-78c4-4a8d-817e-235827d3934f" "344a9889-ff90-4d72-8911-30b72404d577"
-			"3a6205b4-4fa7-4380-ae03-bc596793aef5" "3c3aef36-8bea-4f6b-95c6-503f2075dd7d"
-			"3f252131-6bd9-4ff6-a411-713a3237b121" "428303b1-8c80-42a5-b6e9-c698762b951d"
-			"436ca890-da37-4828-810e-e321b920a213" "445524ef-22d8-4682-9506-93e12dc5d05c"
-			"4477a351-57aa-491d-8d6c-736a198c6920" "473e8952-4e40-4254-ac3b-e3ebb1eb7488"
-			"4a88224e-6035-4cf6-a1db-98d06102f7e5" "4ad88f33-d888-4d58-995a-0c7a34aa7d2e"
-			"509ae6c8-c5fa-45e1-8cda-060c6fe34e23" "59e789a4-91ff-4c7e-8649-71198220f09d"
-			"61a3087e-9c49-4b35-92f2-ae248975b7c5" "62cee386-d17a-4dbf-89bd-f06b432b3be5"
-			"65c23f67-86f6-48ce-aa67-b87304f99b1f" "68907e41-b0ae-400c-ad2a-9451cc251a9e"
-			"6d927956-524f-449a-ae8e-4951c876c20d" "6ed9fd14-6ce1-439a-9ce9-44ac69dc9a7f"
-			"74c5e5b4-e05f-4936-9c97-fa54655c51ea" "79d9da80-8c88-4743-bbdd-624acd2410c4"
-			"7fbce7fe-2f60-4bad-9b97-55a881776bb6" "830b36f0-7323-4806-ab6c-c199843a437c"
-			"8adb6486-138e-463b-9838-3cd0f97a5a7e" "9438ae25-aef3-487b-a5e8-90fffa361f45"
+		(members "009550d5-2990-4ad1-a3d7-d010f3d336c4" "00c08014-d9a6-458d-a25f-47aee30f3706"
+			"05e1108e-6ade-45b6-8ee5-93297f0809cb" "091f30f1-b649-4f01-b896-58e05a611ba3"
+			"094b194e-0616-4f11-b99c-011bcc3eb3d5" "0d7bf8cc-763c-4d73-a79d-c008511989c4"
+			"1030fe69-ed03-412a-a121-e00c15f2cbd9" "11be32db-d326-4050-896b-7b42c8180973"
+			"1525eefc-db0f-4128-b1fe-bcf595bb1ef8" "1763a40e-1121-4ab1-a1e8-7f43c30ca1c7"
+			"1b906849-1e54-4e2a-93c0-fe6b986ff8b7" "221f80ae-7cc2-43bf-a861-1c55bf3d46d6"
+			"2303f457-5b0d-4715-9218-4f59bb6d9517" "27a712fc-486f-424f-8355-7e1d4657289e"
+			"2ed12085-8670-4206-8ce0-7281c614a2e6" "30cca68c-2bc3-4d30-bad8-ec9e12f7a6fb"
+			"3203af40-4d93-4104-aeb6-ea5d71acfc20" "3290ba86-78c4-4a8d-817e-235827d3934f"
+			"344a9889-ff90-4d72-8911-30b72404d577" "3a6205b4-4fa7-4380-ae03-bc596793aef5"
+			"3c3aef36-8bea-4f6b-95c6-503f2075dd7d" "3f252131-6bd9-4ff6-a411-713a3237b121"
+			"428303b1-8c80-42a5-b6e9-c698762b951d" "436ca890-da37-4828-810e-e321b920a213"
+			"445524ef-22d8-4682-9506-93e12dc5d05c" "4477a351-57aa-491d-8d6c-736a198c6920"
+			"473e8952-4e40-4254-ac3b-e3ebb1eb7488" "4a88224e-6035-4cf6-a1db-98d06102f7e5"
+			"4ad88f33-d888-4d58-995a-0c7a34aa7d2e" "509ae6c8-c5fa-45e1-8cda-060c6fe34e23"
+			"59e789a4-91ff-4c7e-8649-71198220f09d" "61a3087e-9c49-4b35-92f2-ae248975b7c5"
+			"62cee386-d17a-4dbf-89bd-f06b432b3be5" "65c23f67-86f6-48ce-aa67-b87304f99b1f"
+			"68907e41-b0ae-400c-ad2a-9451cc251a9e" "6d927956-524f-449a-ae8e-4951c876c20d"
+			"6ed9fd14-6ce1-439a-9ce9-44ac69dc9a7f" "74c5e5b4-e05f-4936-9c97-fa54655c51ea"
+			"79d9da80-8c88-4743-bbdd-624acd2410c4" "7fbce7fe-2f60-4bad-9b97-55a881776bb6"
+			"830b36f0-7323-4806-ab6c-c199843a437c" "8adb6486-138e-463b-9838-3cd0f97a5a7e"
+			"8fe9930c-879c-4391-9f6f-ca2f1acb29f8" "9438ae25-aef3-487b-a5e8-90fffa361f45"
 			"9571156f-28b0-4495-8c8a-9684169dcb68" "9636a53e-0a5b-4c3e-98f4-ae2f3ae54ac5"
 			"9961d2d8-f630-4466-908d-aab376453fa5" "99c26d6b-994f-4655-93f1-bfa20f8024db"
@@
 			"cbd7d602-d38a-4ead-b983-13739a88d44f" "cf61183a-bf4f-45a8-ae85-f06501b4b209"
 			"d3d462ce-fa31-4782-b7b1-a392952e4759" "d5110076-188a-4c6e-a2d1-9a975682ce1c"
-			"d5a75964-896c-4219-85b0-d21bf6ecae49" "dd10a929-d81b-4394-b618-8af2c02047d1"
-			"df199ef3-f181-493c-8de3-50fcda1d4dd9" "e45be571-5de6-4a27-bd2e-a96d9663f0e6"
-			"e72e863d-0273-4df0-a8d0-3cfcdbed76a8" "ef51a9de-38ff-40cb-a8bc-09dbd12d645e"
-			"f1dbf3f1-86a6-4574-adf7-cccbb52d29af" "f2194696-8fdc-44d7-be2e-e8bb02866fc7"
-			"f5d8c6ce-b692-4a95-bb46-83ac27d60f3f" "f860e1f4-1afd-4bb1-bde6-86d9a41d204d"
-			"fc3a355e-a0ba-4424-a118-76e623ba2300"
-		)
-	)
+			"d5a75964-896c-4219-85b0-d21bf6ecae49" "df199ef3-f181-493c-8de3-50fcda1d4dd9"
+			"e45be571-5de6-4a27-bd2e-a96d9663f0e6" "e72e863d-0273-4df0-a8d0-3cfcdbed76a8"
+			"ef51a9de-38ff-40cb-a8bc-09dbd12d645e" "f1dbf3f1-86a6-4574-adf7-cccbb52d29af"
+			"f2194696-8fdc-44d7-be2e-e8bb02866fc7" "f5d8c6ce-b692-4a95-bb46-83ac27d60f3f"
+			"f860e1f4-1afd-4bb1-bde6-86d9a41d204d"
+		)
+	)
